File: single-tube-condensor-schematic/_autosave-single-tube-condensor-schematic.kicad_sch (KiCad schematic)
At the start: 32 parts, among them J1 3-phase-power-connector, K1 relay-SPDT-888-6798, K2 relay-SPDT-888-6798, K3 relay-SPDT-888-6798, K4 Finder-DPDT-relay-DIN, K5 Finder-DPDT-relay-DIN, Q1 IRF540N, SW1 enable-keyswitch, SW2 emergancy-stop-button, SW3 mode-keyswitch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

Commit message: big changes
Parts:
- A3: footprint 000-industrial:adam-6xxx -> 000-industrial:raspberry-pi
Changed lines of the file:
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@@
 			)
 		)
-		(property "Footprint" "000-industrial:adam-6xxx"
+		(property "Footprint" "000-industrial:raspberry-pi"
 			(at 151.13 223.52 0)
 			(effects
